File: ESP32P4C5_Board.kicad_pcb (KiCad board)
At the start: 4 copper layers, 100 x 50 mm, 182 parts, among them IC1 ESP32-C5HR8, J10 UART1_HDR, J11 UART2_HDR, J13 I2C1_Headers, J2 Debug_Pins, J3 SMA PCB END LAUNCH JACK ROUND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, J4 I/O_HDR, J6 USB_C_Receptacle_USB2.0_16P, J7 P4_DEBUG_PINS, J9 USB_C_Receptacle_USB2.0_16P, U1 ESP32-P4NRW16, U11 W25Q256JWPIQ, U14 SN74LVC1G07DBVR, U15 SN74LVC1G07DBVR, U2 USBLC6-2SC6, U4 USBLC6-2SC6, U5 W25Q128JVS, U8 TCA9517D, Y2 ECS-400-10-33B-CKM-TR, Y3 ABM8W-48.0000MHZ-7-B1U-T3

Commit message: Updated notes
Parts:
- removed C17: 1u, Capacitor_SMD:C_0805_2012Metric
- C2, C21, C22, C23, C24, C25, C26, C27, L1, L2, R10, R43, R44, R45, R46, R47, SMPS2: moved to B.Cu
- R35: value 47k -> 1u; footprint Resistor_SMD:R_0603_1608Metric -> Resistor_SMD:R_0805_2012Metric
- R40: value 546R -> 480R
- moved C24 49.6 mm to (130.8, 84.7), turned to 180 degrees
- moved C2 49.4 mm to (131.6, 98.7)
- moved C23 49.1 mm to (131.0, 90.8)
- moved C21 49.1 mm to (130.9, 101.9), turned to 180 degrees
- moved C25 49.0 mm to (130.8, 87.5), turned to 180 degrees
- moved C26 48.8 mm to (122.0, 91.8), turned to 90 degrees
- moved R10 48.6 mm to (129.7, 98.7)
- moved C22 48.5 mm to (130.9, 104.6), turned to 180 degrees
- moved R44 48.5 mm to (129.1, 90.7)
- moved R45 48.4 mm to (128.9, 93.7), turned to 180 degrees
- moved R43 48.4 mm to (128.8, 95.8), turned to 180 degrees
- moved R46 48.1 mm to (126.7, 98.2), turned to 180 degrees
- moved SMPS2 48.1 mm to (125.2, 94.9), turned to 180 degrees
- moved L1 48.1 mm to (126.3, 100.9), turned to 0 degrees
- moved R47 48.1 mm to (126.0, 91.3), turned to 180 degrees
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Connections:
- net /Power_Management/OUT renamed /Power_Management/PWR_C+

Commit message: SMA Update
Parts:
- C14: value 470u -> 1u
- R35: value 1u -> 47k
- moved R16 56.8 mm to (204.2, 65.6)
- moved R23 56.8 mm to (204.2, 68.5)
- moved C19 32.9 mm to (202.0, 139.7)
- moved DI2 32.9 mm to (216.4, 122.0)
- moved R26 32.9 mm to (197.8, 139.9)
- moved R30 32.9 mm to (216.2, 108.6)
- moved R31 32.9 mm to (216.2, 111.6)
- moved U12 32.9 mm to (196.4, 137.2)
- moved U8 32.9 mm to (218.2, 116.4)
- moved R46 5.95 mm to (125.0, 103.9), turned to -90 degrees
- moved R47 5.33 mm to (123.3, 86.8)
- moved R29 3.76 mm to (156.5, 104.4)
- moved R28 3.76 mm to (156.4, 106.6)
- moved C16 2.47 mm to (117.0, 94.1), turned to 90 degrees
- moved RN14 2.40 mm to (161.5, 103.2)
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Connections:
- net /Power_Management/PG renamed /Power_Management/PG_OD
- net Net-(DP1-ANT) renamed /ESP32-C5HR8/ANT
- J2 pad 11: GND -> ESP_3V3
- J7 pad 11: GND -> ESP_3V3
- U1 pad 1: /ESP32-P4NRW16/GPIO1 -> /ESP32-C5HR8/GPIO0
- U1 pad 104: /ESP32-P4NRW16/GPIO0 -> /ESP32-C5HR8/GPIO1
Routing:
- net /ESP32-P4NRW16/GPIO10_SPI2_MISO: track 17.1 -> 70.8 mm, vias 0 -> 2
- net /ESP32-C5HR8/GPIO0: track 9.24 -> 34.3 mm
- net /ESP32-C5HR8/GPIO1: track 9.38 -> 33.5 mm
- net /ESP32-P4NRW16/GPIO2_MTCK: track 2.23 -> 23.7 mm
- net /ESP32-P4NRW16/GPIO3_MTDI: track 2.30 -> 21.6 mm
- net /ESP32-P4NRW16/GPIO4_MTMS: track 2.38 -> 19.5 mm
- net GND: track 45.6 -> 62.4 mm, vias 122 -> 125
- net /ESP32-P4NRW16/GPIO5_MTDO: track 2.45 -> 17.5 mm
- net /Power_Management/PG_OD: track 0.00 -> 14.5 mm
- net /ESP32-C5HR8/GPIO6_SDIO_INT: track 18.0 -> 27.5 mm
- net /ESP32-P4NRW16/GPIO9_SPI2_CK: track 61.9 -> 69.4 mm
- net /ESP32-P4NRW16/GPIO8_SPI2_MOSI: track 60.8 -> 68.0 mm
- net /ESP32-P4NRW16/GPIO39_CDATA0_R: track 4.32 -> 11.0 mm
- net /ESP32-P4NRW16/GPIO40_CDATA1_R: track 4.70 -> 10.7 mm
- net /ESP32-P4NRW16/GPIO41_CDATA2_R: track 4.85 -> 10.5 mm
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- added copper zone on B.Cu, net /Power_Management/EN/UVLO
- added copper zone on B.Cu, net /Power_Management/FB1
- added copper zone on B.Cu, net /Power_Management/OVLO
- added copper zone on B.Cu, net /Power_Management/PGTH
- added copper zone on B.Cu, net /Power_Management/PWR+
- added copper zone on B.Cu, net /Power_Management/PWR_C+
- added copper zone on B.Cu, net /Power_Management/SW1
- added copper zone on B.Cu, net /Power_Management/SW2
- added copper zone on B.Cu, net /Power_Management/TPS62442RQRR_2_FB
- added copper zone on B.Cu, net ESP_VDD_HP
- added copper zone on B.Cu, net PWR_D+

Commit message: QSPI Memory Bus
Parts:
- removed C41, C42: 1uF, Capacitor_SMD:C_0603_1608Metric
- removed FPC4: FPC_BXCONN_FC-10D15P11H25, Personal_Project:FPC_BXCONN_FC-10D15P11H25
- removed J7: P4_DEBUG_PINS, Connector_PinHeader_2.54mm:PinHeader_2x07_P2.54mm_Horizontal
- removed R37: 1k, Resistor_SMD:R_0805_2012Metric_1
- removed R41: 10k, Resistor_SMD:R_0805_2012Metric_1
- removed U10, U6: ~, Personal_Project:Button_SKSCLCE010
- added C17: 100n, Capacitor_SMD:C_0603_1608Metric, B.Cu at (132.3, 72.9)
- added C28: 100n, Capacitor_SMD:C_0603_1608Metric, B.Cu at (141.0, 75.5)
- added C31: 1u, Capacitor_SMD:C_0805_2012Metric, B.Cu at (136.4, 73.5)
- added C38: 18p, Capacitor_SMD:C_0603_1608Metric, F.Cu at (139.1, 77.8)
- added C39: 18p, Capacitor_SMD:C_0603_1608Metric, F.Cu at (135.7, 80.6)
- added C9: 100n, Capacitor_SMD:C_0603_1608Metric, B.Cu at (151.9, 72.6)
- added FPC7: FPC_FPC05-WFB11-22P111-H20, Personal_Project:FPC_FPC05-WFB11-22P111-H20, F.Cu at (128.2, 100.2)
- added IC2: CAN_MCP2518FDT-H_SL, Personal_Project:CAN_MCP2518FDT-H_SL, F.Cu at (146.3, 77.3)
- added IC3: CAN_ATA6563-GAQW1, Personal_Project:CAN_ATA6563_GAQW1, F.Cu at (138.6, 74.0)
- added J1: P4_DEBUG_PINS, Connector_PinHeader_2.54mm:PinHeader_2x06_P2.54mm_Horizontal, F.Cu at (154.7, 77.1)
- added JST1: JST_S3B-XH-2.54, Personal_Project:JST_S3B-XH-SHDRRA3W64P0X250_1X3_990X1150X610P, F.Cu at (130.4, 78.5)
- added R3: 120R, Resistor_SMD:R_0603_1608Metric, F.Cu at (133.9, 74.0)
- added Y1: Crystal_ABM8G-40.000MHZ-18-D2Y-T, Crystal:Crystal_SMD_Abracon_ABM8G-4Pin_3.2x2.5mm, F.Cu at (138.8, 80.5)
- C15: footprint Capacitor_SMD:C_0805_2012Metric -> Capacitor_SMD:C_0603_1608Metric
- C18: value 1uF -> 1u; moved to B.Cu
- DI2, R30, R31, U8: moved to B.Cu
- U11: value W25Q256JWPIQ -> BY25Q128ESSIG(T); footprint Package_SON:WSON-8-1EP_6x5mm_P1.27mm_EP3.4x4.3mm -> Package_SO:SOP-8_5.28x5.23mm_P1.27mm
- U3: value ~ -> LDO_TPS7A2050PDBVR; footprint Personal_Project:Button_SKSCLCE010 -> Personal_Project:LDO_TPS7A2050PDBVR; moved to B.Cu
- moved R31 106.0 mm to (111.8, 129.8), turned to 180 degrees
- moved U8 103.5 mm to (115.7, 102.1), turned to -90 degrees
- moved DI2 101.8 mm to (115.5, 108.2), turned to -90 degrees
- moved R30 95.1 mm to (121.1, 109.5), turned to 180 degrees
- moved U3 82.7 mm to (136.4, 76.9), turned to 90 degrees
- moved J11 61.6 mm to (157.6, 136.2)
- moved FPC3 60.6 mm to (160.2, 46.6)
- moved R19 37.5 mm to (134.9, 113.4)
- moved SP1 37.4 mm to (128.3, 113.3)
- moved C18 34.9 mm to (136.4, 80.3)
- moved R2 33.3 mm to (152.0, 60.1)
- moved FPC5 32.9 mm to (155.8, 149.5)
- moved FPC6 32.2 mm to (141.0, 148.8)
- moved G*** 21.2 mm to (181.7, 108.1)
- moved U15 10.4 mm to (123.4, 83.4), turned to 0 degrees
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Connections:
- net /ESP32-P4NRW16/GPIO24_USB1P1_N0 renamed /ESP32-P4NRW16/USB1P1_N
- net /ESP32-P4NRW16/GPIO25_USB1P1_P0 renamed /ESP32-P4NRW16/USB1P1_P
- net /ESP32-P4NRW16/P4_USB_HS_DM renamed /ESP32-P4NRW16/P4_USB_HS_DN
- net Net-(U1A-GPIO24_USB1P1_N0) renamed /ESP32-P4NRW16/USB1P1_R_N
- net Net-(U1A-GPIO25_USB1P1_P0) renamed /ESP32-P4NRW16/USB1P1_R_P
- C18 pad 2: Net-(C18-Pad2) -> PWR_D+
- FPC2 pad 24: /ESP32-P4NRW16/GPIO7_SPI2_CS -> /ESP32-P4NRW16/GPIO51
- FPC2 pad 26: /ESP32-P4NRW16/GPIO10_SPI2_MISO -> /ESP32-P4NRW16/GPIO52
- FPC2 pad 28: /ESP32-P4NRW16/GPIO9_SPI2_CK -> /ESP32-P4NRW16/GPIO53
- FPC2 pad 30: /ESP32-P4NRW16/GPIO8_SPI2_MOSI -> /ESP32-P4NRW16/GPIO54
- J2 pad 11: ESP_3V3 -> GND
- J2 pad 13: GND -> ESP_3V3
- RN2 pad 1: /ESP32-P4NRW16/GPIO7_SPI2_CS -> /CAN-FD_BUS/NCS
- RN2 pad 2: /ESP32-P4NRW16/GPIO8_SPI2_MOSI -> /CAN-FD_BUS/SDI
- RN2 pad 3: /ESP32-P4NRW16/GPIO9_SPI2_CK -> /CAN-FD_BUS/SCK
- RN2 pad 4: /ESP32-P4NRW16/GPIO10_SPI2_MISO -> /CAN-FD_BUS/SDO
- U1 pad 12: /ESP32-P4NRW16/GPIO11 -> /CAN-FD_BUS/~{_INT0}/GPIO0/XSTBY
- U1 pad 13: /ESP32-P4NRW16/GPIO12 -> /CAN-FD_BUS/~{INT1}/GPIO1
- U1 pad 16: /ESP32-P4NRW16/GPIO15 -> /CAN-FD_BUS/CLKO/SOF
- U1 pad 17: /ESP32-P4NRW16/GPIO16 -> /CAN-FD_BUS/~{INT}
- U3 pad 1: GND -> PWR_D+
- U3 pad 3: /Buttons/USR_BTN0 -> PWR_D+
- U3 pad 4: /Buttons/USR_BTN0 -> unconnected-(U3-NC-Pad4)
Routing:
- net /ESP32-P4NRW16/GPIO10_SPI2_MISO: track 70.8 -> 0.00 mm, vias 2 -> 0
- net /ESP32-P4NRW16/GPIO9_SPI2_CK: track 69.4 -> 0.00 mm, vias 2 -> 0
- net /ESP32-P4NRW16/GPIO8_SPI2_MOSI: track 68.0 -> 0.00 mm, vias 2 -> 0
- net /ESP32-P4NRW16/GPIO7_SPI2_CS: track 62.9 -> 0.00 mm, vias 2 -> 0
- net /ESP32-P4NRW16/P4_USB_HS_DP: track 0.00 -> 52.1 mm
- net /ESP32-P4NRW16/P4_USB_HS_DN: track 0.00 -> 52.0 mm
- net /ESP32-P4NRW16/GPIO17: track 2.84 -> 53.1 mm
- net /ESP32-P4NRW16/GPIO18: track 3.14 -> 51.3 mm
- net /ESP32-P4NRW16/GPIO20: track 3.81 -> 49.1 mm, vias 0 -> 1
- net GND: track 62.4 -> 107.6 mm, vias 125 -> 198
- net /ESP32-P4NRW16/CHIP_PU: track 5.83 -> 49.5 mm, vias 1 -> 2
- net /ESP32-P4NRW16/GPIO21: track 3.78 -> 46.2 mm, vias 0 -> 1
- net /ESP32-P4NRW16/GPIO54: track 7.64 -> 49.6 mm, vias 1 -> 2
- net /ESP32-P4NRW16/GPIO22: track 3.29 -> 43.8 mm, vias 0 -> 1
- net /ESP32-P4NRW16/GPIO14: track 2.75 -> 43.2 mm
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- added copper zone on F.Cu, net /Power_Management/PWR_C+
- added copper zone on B.Cu, net VBUS1+
- added copper zone on F.Cu, net VBUS1+
- added copper zone on B.Cu, net VBUS2+
- added copper zone on F.Cu, net VBUS2+
Other:
- board text added: "3V3"
- board text added: "CAMERA OV5647"
- board text added: "CAN-FD"
- board text added: "GP2-MTCK"
- board text added: "USB1"
- board text added: "USB2"

Commit message: Interface Update
Parts:
- removed FPC5, FPC6: FPC_0545481072, Personal_Project:FPC_10051922_1010
- removed J10: UART1_HDR, Personal_Project:PinHeader_2x03_P2.54mm_Horizontal_Court
- removed J11: UART2_HDR, Personal_Project:PinHeader_2x03_P2.54mm_Horizontal_Court
- removed J4: I/O_HDR, Connector_PinHeader_2.54mm:PinHeader_2x05_P2.54mm_Horizontal
- removed L6: 24n, Inductor_SMD:L_0603_1608Metric
- removed TP1, TP2, TP3, TP4: TestPoint, TestPoint:TestPoint_Pad_1.5x1.5mm
- removed U8: TCA9517D, Package_SO:SOIC-8_3.9x4.9mm_P1.27mm
- added C41: 100n, Capacitor_SMD:C_0603_1608Metric, B.Cu at (147.4, 117.8)
- added G***: LOGO, Personal_Project:PCB_Logo, B.Cu at (190.3, 104.6)
- added R14: 33R, Resistor_SMD:R_0603_1608Metric, B.Cu at (170.2, 81.7)
- added R37: 10k, Resistor_SMD:R_0603_1608Metric, B.Cu at (183.2, 79.5)
- added R4: 0R, Resistor_SMD:R_0603_1608Metric, F.Cu at (180.4, 86.0)
- added R5: 10k, Resistor_SMD:R_0603_1608Metric, B.Cu at (138.0, 117.7)
- added RN6: 33R, Resistor_SMD:R_Array_Convex_4x0402, F.Cu at (160.1, 99.0)
- added SW1: XUNPU DSHP-01-TS-GER, Button_Switch_SMD:SW_DIP_SPSTx01_Slide_Copal_CHS-01B_W7.62mm_P1.27mm, F.Cu at (148.0, 117.8)
- added TP10: TestPoint, TestPoint:TestPoint_Pad_1.5x1.5mm, B.Cu at (164.8, 85.7)
- added TP5: TestPoint, TestPoint:TestPoint_Pad_1.5x1.5mm, B.Cu at (125.5, 115.2)
- added TP6: TestPoint, TestPoint:TestPoint_Pad_1.5x1.5mm, B.Cu at (129.0, 88.0)
- added TP7: TestPoint, TestPoint:TestPoint_Pad_1.5x1.5mm, B.Cu at (120.2, 99.0)
- added TP8: TestPoint, TestPoint:TestPoint_Pad_1.5x1.5mm, B.Cu at (112.8, 88.2)
- added TP9: TestPoint, TestPoint:TestPoint_Pad_1.5x1.5mm, B.Cu at (143.9, 76.3)
- C49, R7, U15: moved to B.Cu
- IC2: value CAN_MCP2518FDT-H_SL -> XINLUDA XLP2518FDT/ESL
- R16, R23: value 33R -> 10k; footprint Resistor_SMD:R_0805_2012Metric -> Resistor_SMD:R_0603_1608Metric; moved to B.Cu
- R28: footprint Resistor_SMD:R_0805_2012Metric_1 -> Resistor_SMD:R_0603_1608Metric
- R29: moved to F.Cu
- R8: value 4k02 -> 4k02_1%
- moved C19 110.9 mm to (102.5, 90.8)
- moved R26 103.8 mm to (105.8, 91.9), turned to 90 degrees
- moved U12 100.7 mm to (104.0, 97.3), turned to 90 degrees
- moved R7 32.3 mm to (158.9, 81.0), turned to 90 degrees
- moved U15 32.3 mm to (155.6, 81.0)
- moved R23 30.4 mm to (177.3, 82.8), turned to 90 degrees
- moved R16 22.2 mm to (186.9, 79.5), turned to 180 degrees
- moved U9 21.9 mm to (159.6, 116.0), turned to 180 degrees
- moved R31 21.6 mm to (112.5, 108.2), turned to 90 degrees
- moved C77 16.2 mm to (160.9, 117.5)
- moved R12 10.4 mm to (117.5, 82.5), turned to 0 degrees
- moved C17 8.89 mm to (141.2, 73.8)
- moved R28 8.58 mm to (152.1, 117.3), turned to -90 degrees
- moved C31 8.27 mm to (142.0, 79.5), turned to -90 degrees
- moved C56 6.81 mm to (149.0, 105.3), turned to -90 degrees
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Connections:
- net Net-(R19-Pad2) renamed /ESP32-P4NRW16/SP+
- C19 pad 2: /ESP32-P4NRW16/CHIP_PU -> /ESP32-C5HR8/RST_PWR
- C23 pad 1: /Power_Management/TPS62442RQRR_2_FB -> /ESP32-P4NRW16/FB_DCDC
- DI2 pad 1: /Interfaces/SCLB -> /ESP32-P4NRW16/GPIO18
- DI2 pad 2: /Interfaces/SDAB -> /ESP32-P4NRW16/GPIO17
- FPC1 pad 2: /Interfaces/SPI_MOSI -> /ESP32-P4NRW16/GPIO20_SPI_MOSI
- FPC1 pad 4: /Interfaces/SPI_MISO -> /ESP32-P4NRW16/GPIO21_SPI_MISO
- FPC1 pad 7: /Interfaces/SPI_CLK -> /ESP32-P4NRW16/GPIO22_SPI_CLK
- FPC1 pad 9: /Interfaces/SPI_CS -> /ESP32-P4NRW16/GPIO23_SPI_CS
- FPC2 pad 20: /ESP32-P4NRW16/GPIO49_PARLIO -> /ESP32-P4NRW16/GPIO48_PARLIO
- FPC2 pad 22: /ESP32-P4NRW16/GPIO48_PARLIO -> /ESP32-P4NRW16/GPIO49_PARLIO
- J1 pad 12: /ESP32-P4NRW16/GPIO14 -> GND
- J1 pad 2: /ESP32-P4NRW16/GPIO37_BOOTM_UART0_TXD -> GND
- J1 pad 4: /ESP32-P4NRW16/GPIO38_BOOTM_UART0_RXD -> GND
- J13 pad 1: /Interfaces/SDAB -> /ESP32-P4NRW16/GPIO17
- J13 pad 2: GND -> /ESP32-P4NRW16/GPIO37_BOOTM_UART0_TXD
- J13 pad 5: /Interfaces/SCLB -> /ESP32-P4NRW16/GPIO18
- J13 pad 6: GND -> /ESP32-P4NRW16/GPIO38_BOOTM_UART0_RXD
- J2 pad 1: GND -> ESP_3V3
- J2 pad 13: ESP_3V3 -> GND
- J2 pad 2: /ESP32-C5HR8/CHIP_PU -> GND
- J2 pad 5: GND -> /ESP32-C5HR8/CHIP_PU
- J2 pad 8: /ESP32-C5HR8/MTDO -> /ESP32-C5HR8/MTDO_R
- R16 pad 1: /Interfaces/UART2_TX/RX -> ESP_3V3
- R16 pad 2: /Interfaces/UART2_TX/RX_R -> /ESP32-C5HR8/MTDI
- R19 pad 1: unconnected-(R19-Pad1) -> /ESP32-P4NRW16/GPIO16
- R23 pad 1: /Interfaces/UART1_TX/RX -> ESP_3V3
- R23 pad 2: /Interfaces/UART1_TX/RX_R -> /ESP32-C5HR8/MTMS
- R26 pad 2: /ESP32-P4NRW16/CHIP_PU -> /ESP32-C5HR8/RST_PWR
- R30 pad 2: /Interfaces/I2C_SDA_HDR -> /ESP32-P4NRW16/GPIO17
- R31 pad 2: /Interfaces/I2C_SCL_HDR -> /ESP32-P4NRW16/GPIO18
- R44 pad 2: /Power_Management/TPS62442RQRR_2_FB -> /ESP32-P4NRW16/FB_DCDC
- R45 pad 1: /Power_Management/TPS62442RQRR_2_FB -> /ESP32-P4NRW16/FB_DCDC
- RN5 pad 1: GND -> /ESP32-P4NRW16/GPIO43_CCLK_R
- RN5 pad 2: /ESP32-P4NRW16/GPIO43_CCLK_R -> GND
- RN5 pad 7: /ESP32-C5HR8/GPIO9_SDIO_CLK -> GND
- RN5 pad 8: GND -> /ESP32-C5HR8/GPIO9_SDIO_CLK
- SMPS2 pad 1: /Power_Management/TPS62442RQRR_2_FB -> /ESP32-P4NRW16/FB_DCDC
- SMPS2 pad 10: /Power_Management/TPS62442RQRR_2_EN -> /ESP32-P4NRW16/EN_DCDC
- U1 pad 15: /ESP32-P4NRW16/GPIO14 -> /CAN-FD_BUS/CLKO/SOF
- U1 pad 16: /CAN-FD_BUS/CLKO/SOF -> /CAN-FD_BUS/~{INT}
- U1 pad 17: /CAN-FD_BUS/~{INT} -> /ESP32-P4NRW16/GPIO16
- U1 pad 22: /ESP32-P4NRW16/GPIO20 -> /ESP32-P4NRW16/GPIO20_SPI_MOSI
- U1 pad 23: /ESP32-P4NRW16/GPIO21 -> /ESP32-P4NRW16/GPIO21_SPI_MISO
- U1 pad 24: /ESP32-P4NRW16/GPIO22 -> /ESP32-P4NRW16/GPIO22_SPI_CLK
- U1 pad 25: /ESP32-P4NRW16/GPIO23 -> /ESP32-P4NRW16/GPIO23_SPI_CS
- U1 pad 89: /ESP32-P4NRW16/GPIO47_PARLIO -> /ESP32-P4NRW16/GPIO47_PARLIO_R
- U1 pad 90: /ESP32-P4NRW16/GPIO48_PARLIO -> /ESP32-P4NRW16/GPIO48_PARLIO_R
- U1 pad 92: /ESP32-P4NRW16/GPIO49_PARLIO -> /ESP32-P4NRW16/GPIO49_PARLIO_R
- U12 pad 3: /ESP32-P4NRW16/CHIP_PU -> /ESP32-C5HR8/RST_PWR
- U12 pad 4: /ESP32-P4NRW16/CHIP_PU -> /ESP32-C5HR8/RST_PWR
Routing:
- net ESP_3V3: track 88.4 -> 218.5 mm, vias 17 -> 36
- net /ESP32-C5HR8/RST_PWR: track 12.4 -> 118.7 mm, vias 0 -> 2
- net /ESP32-P4NRW16/GPIO20_SPI_MOSI: track 0.00 -> 85.3 mm, vias 0 -> 2
- net /ESP32-P4NRW16/GPIO21_SPI_MISO: track 0.00 -> 85.3 mm, vias 0 -> 2
- net /ESP32-P4NRW16/GPIO23_SPI_CS: track 0.00 -> 85.3 mm, vias 0 -> 2
- net /ESP32-P4NRW16/GPIO22_SPI_CLK: track 0.00 -> 85.2 mm, vias 0 -> 2
- net /ESP32-P4NRW16/FB_DCDC: track 0.40 -> 80.2 mm, vias 0 -> 5
- net GND: track 107.6 -> 183.8 mm, vias 198 -> 494
- net /ESP32-P4NRW16/EN_DCDC: track 0.72 -> 73.8 mm, vias 0 -> 5
- net /ESP32-P4NRW16/GPIO16: track 0.00 -> 70.6 mm, vias 0 -> 2
- net /ESP32-P4NRW16/GPIO38_BOOTM_UART0_RXD: track 2.52 -> 57.5 mm, vias 0 -> 2
- net /ESP32-P4NRW16/GPIO20: track 49.1 -> 0.00 mm, vias 1 -> 0
- net /ESP32-P4NRW16/GPIO21: track 46.2 -> 0.00 mm, vias 1 -> 0
- net /ESP32-P4NRW16/GPIO37_BOOTM_UART0_TXD: track 2.68 -> 47.7 mm, vias 0 -> 2
- net /ESP32-P4NRW16/GPIO22: track 43.8 -> 0.00 mm, vias 1 -> 0
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- added copper zone on B.Cu, net /ESP32-P4NRW16/FB_DCDC
- added copper zone on F.Cu, net /ESP32-P4NRW16/SP+
- added copper zone on B.Cu, net 5V+
- added copper zone on B.Cu, net ESP_FLASH
- added copper zone on B.Cu, net ESP_LDO_VDDO_3
- added copper zone on B.Cu, net ESP_LDO_VDDO_4
- added copper zone on B.Cu, net ESP_LDO_VDDO_PSRAM
- added copper zone on F.Cu, net ESP_VDD_HP
- removed copper zone on B.Cu, net /Power_Management/TPS62442RQRR_2_FB
Other:
- board text added: "BOOTM"
- board text added: "CK"
- board text added: "DI"
- board text added: "DO"
- board text added: "ESP32P4C5 BOARD Revision: REV A Designer: Peter Hancak MCU: ESP32P4, ESP32C5 SMPS: TPS62442RQRR VIN: 5V to 5.5V"
- board text added: "G"
- board text added: "G13"
- board text added: "G2-MCK"
- board text added: "G3-MDI"
- board text added: "G4-MMS"
- board text added: "G5-MO"
- board text added: "GND"
- board text added: "H"
- board text added: "JTAG SRC"
- board text added: "L"
- board text added: "MS"
- board text added: "PU"
- board text added: "RST"
- board text added: "RX"
- board text added: "TX"
- board text added: "USB/PINS"
- board text removed: "GP2-MTCK"
