File: ESP32P4C5_Board.kicad_pcb (KiCad board)
At the start: 4 copper layers, 100 x 50 mm, 189 parts, among them IC1 ESP32-C5HR8, IC2 XINLUDA XLP2518FDT/ESL, IC3 CAN_ATA6563-GAQW1, J1 P4_DEBUG_PINS, J13 I2C1_Headers, J2 Debug_Pins, J3 SMA PCB END LAUNCH JACK ROUND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, J6 USB_C_Receptacle_USB2.0_16P, J9 USB_C_Receptacle_USB2.0_16P, SW1 XUNPU DSHP-01-TS-GER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

Commit message: Update
Parts:
- removed C1, C5: 2p, Capacitor_SMD:C_0603_1608Metric
- removed C6, C7: 1p, Capacitor_SMD:C_0603_1608Metric
- removed L4: 2n8, Inductor_SMD:L_0603_1608Metric
- removed L5: 2n, Inductor_SMD:L_0603_1608Metric
Connections:
- DP1 pad 4: /ESP32-C5HR8/ANT_5G -> /ESP32-C5HR8/ANT_5G_M
- DP1 pad 6: /ESP32-C5HR8/ANT_2G -> /ESP32-C5HR8/ANT_2G_M
Routing:
- net /ESP32-C5HR8/ANT_2G: track 5.44 -> 0.00 mm
- net /ESP32-C5HR8/ANT_2G_M: track 4.39 -> 9.82 mm
- net /ESP32-C5HR8/ANT_5G: track 5.20 -> 0.00 mm
- net GND: track 183.8 -> 186.3 mm, vias 494 -> 497
- net /ESP32-C5HR8/ANT_5G_M: track 6.48 -> 7.24 mm
- added copper zone on F.Cu, net /ESP32-C5HR8/ANT_2G_M
- added copper zone on F.Cu, net /ESP32-C5HR8/ANT_5G_M
- removed copper zone on F.Cu, net /ESP32-C5HR8/ANT_2G
- removed copper zone on F.Cu, net /ESP32-C5HR8/ANT_5G
