File: ESP32P4C5_Board.kicad_pcb (KiCad board)
At the start: 4 copper layers, 100 x 50 mm, 188 parts, among them IC1 ESP32-C5HR8, IC2 XINLUDA XLP2518FDT/ESL, IC3 CAN_ATA6563-GAQW1, J1 P4_DEBUG_PINS, J13 I2C1_Headers, J2 Debug_Pins, J3 SMA PCB END LAUNCH JACK ROUND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, J6 USB_C_Receptacle_USB2.0_16P, J9 USB_C_Receptacle_USB2.0_16P, SW1 XUNPU DSHP-01-TS-GER, U11 BY25Q128ESSIG(T), U14 SN74LVC1G07DBVR, U15 SN74LVC1G07DBVR, U2 USBLC6-2SC6, U3 ESP32-P4NRW32X, U4 USBLC6-2SC6, U5 W25Q128JVS, U6 SMPS_TPS63002DRCR, Y1 Crystal_ABM8G-40.000MHZ-18-D2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, Y2 ECS-400-10-33B-CKM-TR, Y3 ABM8W-48.0000MHZ-7-B1U-T3

Commit message: ESP32P4_Fix
Parts:
- removed JST1: JST_S3B-XH-2.54, Personal_Project:JST_S3B-XH-SHDRRA3W64P0X250_1X3_990X1150X610P
- added J4: CAN_HDR, Connector_PinHeader_2.54mm:PinHeader_1x03_P2.54mm_Horizontal, F.Cu at (125.4, 78.5)
Other:
- board text added: "CAN-BUS"
