File: ESP32-C5HR8.kicad_sch (KiCad schematic)
At the start: 40 parts, among them IC1 ESP32-C5HR8, J2 Debug_Pins, J3 SMA PCB END LAUNCH JACK ROUND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, U14 SN74LVC1G07DBVR, U5 W25Q128JVS, Y3 ABM8W-48.0000MHZ-7-B1U-T3

Commit message: SMA Update
Connections:
- net ESP_3V3: now also J2.11 (Pin_11)
- net GND: no longer J2.11 (Pin_11)
- net ANT: now reaches DP1.2 (ANT), J3.3 (Signal)
Changed lines of the file:
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@@
 	)
 	(junction
-		(at 34.29 45.72)
-		(diameter 0)
-		(color 0 0 0 0)
-	)
-	(junction
 		(at 199.39 81.28)
 		(diameter 0)
@@
 	(wire
 		(pts
+			(xy 30.48 45.72) (xy 30.48 44.45)
+		)
+		(stroke
+			(width 0)
+			(type default)
+		)
+	)
+	(wire
+		(pts
 			(xy 241.3 123.19) (xy 241.3 142.24)
 		)
@@
 	(wire
 		(pts
-			(xy 34.29 45.72) (xy 38.1 45.72)
-		)
-		(stroke
-			(width 0)
-			(type default)
-		)
-	)
-	(wire
-		(pts
 			(xy 43.18 168.91) (xy 29.21 168.91)
 		)
@@
 	(wire
 		(pts
-			(xy 34.29 45.72) (xy 34.29 48.26)
+			(xy 34.29 43.18) (xy 34.29 48.26)
 		)
 		(stroke
@@
 	(wire
 		(pts
-			(xy 222.25 44.45) (xy 234.95 44.45)
+			(xy 38.1 45.72) (xy 30.48 45.72)
 		)
 		(stroke
@@
 	(wire
 		(pts
-			(xy 154.94 48.26) (xy 154.94 73.66)
+			(xy 222.25 44.45) (xy 234.95 44.45)
 		)
 		(stroke
@@
 	(wire
 		(pts
-			(xy 261.62 123.19) (xy 261.62 125.73)
+			(xy 154.94 48.26) (xy 154.94 73.66)
 		)
 		(stroke
@@
 	(wire
 		(pts
-			(xy 279.4 111.76) (xy 279.4 114.3)
+			(xy 261.62 123.19) (xy 261.62 125.73)
 		)
 		(stroke
@@
 	(wire
 		(pts
-			(xy 95.25 83.82) (xy 97.79 83.82)
+			(xy 279.4 111.76) (xy 279.4 114.3)
 		)
 		(stroke
@@
 	(wire
 		(pts
-			(xy 229.87 139.7) (xy 232.41 139.7)
+			(xy 95.25 83.82) (xy 97.79 83.82)
 		)
 		(stroke
@@
 	(wire
 		(pts
-			(xy 36.83 96.52) (xy 57.15 96.52)
+			(xy 229.87 139.7) (xy 232.41 139.7)
 		)
 		(stroke
@@
 	(wire
 		(pts
-			(xy 34.29 43.18) (xy 34.29 45.72)
+			(xy 36.83 96.52) (xy 57.15 96.52)
 		)
 		(stroke
@@
 		)
 	)
+	(label "ANT"
+		(at 200.66 139.7 180)
+		(effects
+			(font
+				(size 1.27 1.27)
+			)
+			(justify right bottom)
+		)
+	)
 	(label "GPIO8_SDIO_DATA0"
 		(at 36.83 91.44 0)
@@
 					(unit 1)
 				)
+			)
+		)
+	)
+	(symbol
+		(lib_id "power:+3.3V")
+		(at 30.48 44.45 0)
+		(mirror y)
+		(unit 1)
+		(exclude_from_sim no)
+		(in_bom yes)
+		(on_board yes)
+		(dnp no)
+		(property "Reference" "#PWR060"
+			(at 30.48 48.26 0)
+			(effects
+				(font
+					(size 1.27 1.27)
+				)
+				(hide yes)
+			)
+		)
+		(property "Value" "ESP_3V3"
+			(at 27.94 40.386 90)
+			(effects
+				(font
+					(size 1.27 1.27)
+				)
+			)
+		)
+		(property "Footprint" ""
+			(at 30.48 44.45 0)
+			(effects
+				(font
+					(size 1.27 1.27)
+				)
+				(hide yes)
+			)
+		)
+		(property "Datasheet" ""
+			(at 30.48 44.45 0)
+			(effects
+				(font
+					(size 1.27 1.27)
+				)
+				(hide yes)
+			)
+		)
+		(property "Description" "Power symbol creates a global label with name \"+3.3V\""
+			(at 30.48 44.45 0)
+			(effects
+				(font
+					(size 1.27 1.27)
+				)
+				(hide yes)
+			)
+		)
+		(pin "1"
+		)
+		(instances
+			(project "ESP32P4C5_Board"
+				(path "/d4a17687-8854-438f-9913-a6ddcff1a679/e64b2c4a-3136-4c33-ae85-e0f033842593"
+					(reference "#PWR060")
+					(unit 1)
+				)

Commit message: QSPI Memory Bus
Connections:
- net ESP_3V3: now also J2.13 (Pin_13); no longer J2.11 (Pin_11)
- net GND: now also J2.11 (Pin_11); no longer J2.13 (Pin_13)
Changed lines of the file:
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@@
 	)
 	(junction
-		(at 34.29 48.26)
-		(diameter 0)
-		(color 0 0 0 0)
-	)
-	(junction
 		(at 279.4 114.3)
 		(diameter 0)
@@
 	)
 	(junction
+		(at 34.29 45.72)
+		(diameter 0)
+		(color 0 0 0 0)
+	)
+	(junction
 		(at 34.29 40.64)
 		(diameter 0)
@@
 	(wire
 		(pts
-			(xy 30.48 45.72) (xy 30.48 44.45)
+			(xy 30.48 46.99) (xy 30.48 48.26)
 		)
 		(stroke
@@
 	(wire
 		(pts
+			(xy 34.29 45.72) (xy 38.1 45.72)
+		)
+		(stroke
+			(width 0)
+			(type default)
+		)
+	)
+	(wire
+		(pts
 			(xy 247.65 142.24) (xy 251.46 142.24)
 		)
@@
 	(wire
 		(pts
+			(xy 34.29 45.72) (xy 34.29 50.8)
+		)
+		(stroke
+			(width 0)
+			(type default)
+		)
+	)
+	(wire
+		(pts
 			(xy 107.95 162.56) (xy 105.41 162.56)
 		)
@@
 	(wire
 		(pts
-			(xy 34.29 43.18) (xy 34.29 48.26)
+			(xy 34.29 43.18) (xy 34.29 45.72)
 		)
 		(stroke
@@
 	(wire
 		(pts
-			(xy 34.29 48.26) (xy 34.29 50.8)
-		)
-		(stroke
-			(width 0)
-			(type default)
-		)
-	)
-	(wire
-		(pts
 			(xy 149.86 48.26) (xy 149.86 73.66)
 		)
@@
 	(wire
 		(pts
-			(xy 38.1 45.72) (xy 30.48 45.72)
-		)
-		(stroke
-			(width 0)
-			(type default)
-		)
-	)
-	(wire
-		(pts
 			(xy 222.25 44.45) (xy 234.95 44.45)
 		)
@@
 	(wire
 		(pts
+			(xy 30.48 48.26) (xy 38.1 48.26)
+		)
+		(stroke
+			(width 0)
+			(type default)
+		)
+	)
+	(wire
+		(pts
 			(xy 67.31 124.46) (xy 67.31 127)
 		)
@@
 	(wire
 		(pts
-			(xy 34.29 48.26) (xy 38.1 48.26)
-		)
-		(stroke
-			(width 0)
-			(type default)
-		)
-	)
-	(wire
-		(pts
 			(xy 30.48 143.51) (xy 39.37 143.51)
 		)
@@
 	(label "ANT"
 		(at 200.66 139.7 180)
+		(fields_autoplaced yes)
 		(effects
 			(font
@@
 	(symbol
 		(lib_id "power:+3.3V")
-		(at 30.48 44.45 0)
+		(at 30.48 46.99 0)
 		(mirror y)
 		(unit 1)
@@
 		(dnp no)
 		(property "Reference" "#PWR060"
-			(at 30.48 48.26 0)
+			(at 30.48 50.8 0)
 			(effects
 				(font
@@
 		)
 		(property "Value" "ESP_3V3"
-			(at 27.94 40.386 90)
+			(at 27.94 42.926 90)
 			(effects
 				(font
@@
 		)
 		(property "Footprint" ""
-			(at 30.48 44.45 0)
+			(at 30.48 46.99 0)
 			(effects
 				(font
@@
 		)
 		(property "Datasheet" ""
-			(at 30.48 44.45 0)
+			(at 30.48 46.99 0)
 			(effects
 				(font
@@
 		)
 		(property "Description" "Power symbol creates a global label with name \"+3.3V\""
-			(at 30.48 44.45 0)
+			(at 30.48 46.99 0)
 			(effects
 				(font

Commit message: Interface Update
Parts:
- removed L6: 24n, Inductor_SMD:L_0603_1608Metric, symbol Device:L
- added R14: 33R, Resistor_SMD:R_0603_1608Metric, symbol Device:R
- added R16, R23, R37: 10k, Resistor_SMD:R_0603_1608Metric, symbol Device:R
- added R4: 0R, Resistor_SMD:R_0603_1608Metric, symbol Device:R
Connections:
- net CHIP_PU: now also J2.5 (Pin_5); no longer J2.2 (Pin_2)
- net ESP_3V3: now also J2.1 (Pin_1), R16.1, R23.1; no longer J2.13 (Pin_13)
- net GND: now also J2.13 (Pin_13), J2.2 (Pin_2), R37.2; no longer J2.1 (Pin_1), J2.5 (Pin_5)
- net MTCK: now also R37.1
- net MTDI: now also R16.2
- net MTDO: now also R14.2; no longer J2.8 (Pin_8)
- net MTMS: now also R23.2
- net at IC1.5 (XTAL_P): now also R4.1
- net at C83.1, Y3.1: now also R4.2
- new net MTDO_R: J2.8 (Pin_8), R14.1
- no-connect marks 4 -> 5
Other:
- note removed: "VDDA Analog Power Supply"
- company: (none) -> Peter Hancak
- title: (none) -> ESP32P4C5_BOARD
- moved on the sheet: C20, C90, J2, JP1, R22, R27, R42, U13, U5

Commit message: Update
Parts:
- removed C1, C5: 2p, Capacitor_SMD:C_0603_1608Metric, symbol Device:C
- removed C6, C7: 1p, Capacitor_SMD:C_0603_1608Metric, symbol Device:C
- removed L4: 2n8, Inductor_SMD:L_0603_1608Metric, symbol Device:L
- removed L5: 2n, Inductor_SMD:L_0603_1608Metric, symbol Device:L
Connections:
- net ANT_2G is gone; now on net ANT_2G_M: DP1.6 (LO-BAND)
- net ANT_5G is gone; now on net ANT_5G_M: DP1.4 (HI-BAND)
Other:
- note removed: "MURATA GQM"
