File: ESP32-C5HR8.kicad_sch (KiCad schematic)
At the start: 44 parts, among them IC1 ESP32-C5HR8, J2 Debug_Pins, J3 SMA PCB END LAUNCH JACK ROUND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, U14 SN74LVC1G07DBVR, U5 W25Q128JVS, Y3 ABM8W-48.0000MHZ-7-B1U-T3

Commit message: C5 RF Update
Parts:
- added C31: 0p3, Capacitor_SMD:C_0402_1005Metric, symbol Device:C
- C30: value 2p6 -> 0p3; footprint Capacitor_SMD:C_0603_1608Metric -> Capacitor_SMD:C_0402_1005Metric
Connections:
- net GND: now also C31.2
- net VDDA1: now also C31.1
Other:
- note added: "BLM21PG601SH1D"
- note added: "Original Cap: One 2p6"
Changed lines of the file:
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@@
 		)
 	)
+	(text "BLM21PG601SH1D"
+		(exclude_from_sim no)
+		(at 235.966 109.728 0)
+		(effects
+			(font
+				(size 1.27 1.27)
+			)
+		)
+	)
 	(text "Internal Low-Dropout (LDO) regulators and the \nPower Amplifier (PA) for the 2.4 GHz and 5 GHz radio."
 		(exclude_from_sim no)
@@
 		)
 	)
+	(text "Original Cap: One 2p6"
+		(exclude_from_sim no)
+		(at 197.358 115.062 0)
+		(effects
+			(font
+				(size 1 1)
+			)
+			(justify left)
+		)
+	)
 	(text "Use Internal 32K"
 		(exclude_from_sim no)
@@
 	)
 	(junction
+		(at 217.17 113.03)
+		(diameter 0)
+		(color 0 0 0 0)
+	)
+	(junction
 		(at 245.11 31.75)
 		(diameter 0)
@@
 	)
 	(junction
-		(at 212.09 101.6)
-		(diameter 0)
-		(color 0 0 0 0)
-	)
-	(junction
 		(at 247.65 123.19)
 		(diameter 0)
@@
 	)
 	(junction
+		(at 199.39 101.6)
+		(diameter 0)
+		(color 0 0 0 0)
+	)
+	(junction
 		(at 124.46 43.18)
 		(diameter 0)
@@
 	)
 	(junction
+		(at 207.01 101.6)
+		(diameter 0)
+		(color 0 0 0 0)
+	)
+	(junction
 		(at 110.49 43.18)
 		(diameter 0)
@@
 	(wire
 		(pts
+			(xy 207.01 101.6) (xy 207.01 104.14)
+		)
+		(stroke
+			(width 0)
+			(type default)
+		)
+	)
+	(wire
+		(pts
 			(xy 154.94 48.26) (xy 149.86 48.26)
 		)
@@
 	(wire
 		(pts
-			(xy 212.09 101.6) (xy 181.61 101.6)
-		)
-		(stroke
-			(width 0)
-			(type default)
-		)
-	)
-	(wire
-		(pts
 			(xy 57.15 77.47) (xy 57.15 96.52)
 		)
@@
 	(wire
 		(pts
+			(xy 217.17 114.3) (xy 217.17 113.03)
+		)
+		(stroke
+			(width 0)
+			(type default)
+		)
+	)
+	(wire
+		(pts
 			(xy 147.32 20.32) (xy 245.11 20.32)
 		)
@@
 	(wire
 		(pts
-			(xy 110.49 54.61) (xy 110.49 55.88)
+			(xy 207.01 113.03) (xy 217.17 113.03)
 		)
 		(stroke
@@
 	(wire
 		(pts
-			(xy 144.78 16.51) (xy 144.78 73.66)
+			(xy 110.49 54.61) (xy 110.49 55.88)
 		)
 		(stroke
@@
 	(wire
 		(pts
-			(xy 149.86 130.81) (xy 149.86 119.38)
+			(xy 144.78 16.51) (xy 144.78 73.66)
 		)
 		(stroke
@@
 	(wire
 		(pts
-			(xy 182.88 48.26) (xy 182.88 50.8)
+			(xy 149.86 130.81) (xy 149.86 119.38)
 		)
 		(stroke
@@
 	(wire
 		(pts
-			(xy 224.79 78.74) (xy 224.79 91.44)
+			(xy 182.88 48.26) (xy 182.88 50.8)
 		)
 		(stroke
@@
 	(wire
 		(pts
-			(xy 212.09 101.6) (xy 217.17 101.6)
+			(xy 224.79 78.74) (xy 224.79 91.44)
 		)
 		(stroke
@@
 	(wire
 		(pts
+			(xy 199.39 101.6) (xy 181.61 101.6)
+		)
+		(stroke
+			(width 0)
+			(type default)
+		)
+	)
+	(wire
+		(pts
 			(xy 217.17 111.76) (xy 217.17 113.03)
 		)
@@
 	(wire
 		(pts
+			(xy 207.01 101.6) (xy 217.17 101.6)
+		)
+		(stroke
+			(width 0)
+			(type default)
+		)
+	)
+	(wire
+		(pts
 			(xy 279.4 99.06) (xy 279.4 101.6)
 		)
@@
 	(wire
 		(pts
+			(xy 207.01 111.76) (xy 207.01 113.03)
+		)
+		(stroke
+			(width 0)
+			(type default)
+		)
+	)
+	(wire
+		(pts
 			(xy 247.65 91.44) (xy 247.65 92.71)
 		)
@@
 	(wire
 		(pts
-			(xy 212.09 101.6) (xy 212.09 104.14)
+			(xy 199.39 101.6) (xy 199.39 104.14)
 		)
 		(stroke
@@
 	(wire
 		(pts
-			(xy 212.09 104.14) (xy 181.61 104.14)
+			(xy 199.39 101.6) (xy 207.01 101.6)
+		)
+		(stroke
+			(width 0)
+			(type default)
+		)
+	)
+	(wire
+		(pts
+			(xy 199.39 104.14) (xy 181.61 104.14)
 		)
 		(stroke
@@
 			)
 		)
-		(property "Value" "2p6"
+		(property "Value" "0p3"
 			(at 217.932 110.49 0)
 			(show_name no)
@@
 			)
 		)
-		(property "Footprint" "Capacitor_SMD:C_0603_1608Metric"
+		(property "Footprint" "Capacitor_SMD:C_0402_1005Metric"
 			(at 218.1352 111.76 0)
 			(hide yes)
@@
 	(symbol
 		(lib_id "power:GND")
-		(at 217.17 113.03 0)
+		(at 217.17 114.3 0)
 		(unit 1)
 		(body_style 1)
@@
 		(dnp no)
 		(property "Reference" "#PWR087"
-			(at 217.17 119.38 0)
+			(at 217.17 120.65 0)
 			(hide yes)
 			(show_name no)
@@
 		)
 		(property "Value" "GND"
-			(at 216.662 117.856 0)
+			(at 216.662 119.126 0)
 			(hide yes)
 			(show_name no)
@@
 		)
 		(property "Footprint" ""
-			(at 217.17 113.03 0)
+			(at 217.17 114.3 0)
 			(hide yes)
 			(show_name no)
@@
 		)
 		(property "Datasheet" ""
-			(at 217.17 113.03 0)
+			(at 217.17 114.3 0)
 			(hide yes)
 			(show_name no)
@@
 		)
 		(property "Description" "Power symbol creates a global label with name \"GND\" , ground"
-			(at 217.17 113.03 0)
+			(at 217.17 114.3 0)
 			(hide yes)
 			(show_name no)
@@
 					(unit 1)
 				)
+			)
+		)
+	)
+	(symbol
+		(lib_id "Device:C")
+		(at 207.01 107.95 0)
+		(unit 1)
+		(body_style 1)
+		(exclude_from_sim no)
+		(in_bom yes)
+		(on_board yes)
+		(in_pos_files yes)
+		(dnp no)
+		(property "Reference" "C31"
+			(at 207.772 105.41 0)
+			(show_name no)
+			(do_not_autoplace no)
+			(effects
+				(font
+					(size 1.27 1.27)
+				)
+				(justify left)
+			)
+		)
+		(property "Value" "0p3"
+			(at 207.772 110.49 0)
+			(show_name no)
+			(do_not_autoplace no)
+			(effects
+				(font
+					(size 1.27 1.27)
+				)
+				(justify left)
+			)
+		)
+		(property "Footprint" "Capacitor_SMD:C_0402_1005Metric"
+			(at 207.9752 111.76 0)
+			(hide yes)
+			(show_name no)
+			(do_not_autoplace no)
+			(effects
+				(font
+					(size 1.27 1.27)
+				)
+			)
+		)
+		(property "Datasheet" ""
+			(at 207.01 107.95 0)
+			(hide yes)
+			(show_name no)
+			(do_not_autoplace no)
+			(effects
+				(font
+					(size 1.27 1.27)
+				)
+			)
+		)
+		(property "Description" "Unpolarized capacitor"
+			(at 207.01 107.95 0)
+			(hide yes)
+			(show_name no)
+			(do_not_autoplace no)
+			(effects
+				(font
+					(size 1.27 1.27)
+				)
+			)
+		)
+		(pin "1"
+		)
+		(pin "2"
+		)
+		(instances
+			(project "ESP32P4C5_Board"
+				(path "/d4a17687-8854-438f-9913-a6ddcff1a679/e64b2c4a-3136-4c33-ae85-e0f033842593"
+					(reference "C31")
+					(unit 1)
+				)

Commit message: RF Update
Parts:
- C35: value 10n_GRM188R72A103KA01 -> 10n_GRM1555C1E103JE01; footprint Capacitor_SMD:C_0603_1608Metric -> Capacitor_SMD:C_0402_1005Metric
- C37: value 10u_GRM188Z71A106KA73 -> 1u_GRM188C71A105MA12
- C6, C7, C89, C92, C93, C94: footprint Capacitor_SMD:C_0603_1608Metric -> Capacitor_SMD:C_0402_1005Metric
- R4: footprint Resistor_SMD:R_0603_1608Metric -> Resistor_SMD:R_0402_1005Metric
- R6: footprint Resistor_SMD:R_0805_2012Metric -> Resistor_SMD:R_0603_1608Metric
Other:
- moved on the sheet: C91, C92, C93

Commit message: RF_Layout
Parts:
- removed C1: 1p, Capacitor_SMD:C_0603_1608Metric, symbol Device:C
- removed C5: 0p6, Capacitor_SMD:C_0603_1608Metric, symbol Device:C
- removed C6: 0p3, Capacitor_SMD:C_0402_1005Metric, symbol Device:C
- removed C7: 0p4, Capacitor_SMD:C_0402_1005Metric, symbol Device:C
- removed DP1: DIPLEXER_DPX205950DT-9026A1, Personal_Project:DIPLEXER_DPX205950DT-9026A1, symbol Personal_Projects:DIPLEXER_DPX205950DT-9026A1
- removed J3: SMA PCB END LAUNCH JACK ROUND PO, Personal_Project:SMA Clip Mount Adapter (top), symbol Personal_Projects:SMA PCB END LAUNCH JACK ROUND PO
- removed L4: 2n4, Inductor_SMD:L_0603_1608Metric, symbol Device:L
- removed L5: 1n3, Inductor_SMD:L_0402_1005Metric_Pad0.77x0.64mm_HandSolder, symbol Device:L
- C37: footprint Capacitor_SMD:C_0603_1608Metric -> Capacitor_SMD:C_0402_1005Metric
- C90: footprint Capacitor_SMD:C_0805_2012Metric -> Capacitor_SMD:C_0603_1608Metric
Other:
- note added: "CQ0402BRNPO0BNR60 CQ series from Yageo"
- note removed: "(40 ~ 45)+j0 (2.4 GHz)"
- note removed: "(50 ~ 65)+j0 (5 GHz)"
- note removed: "All traces at 50 Ohm"
- note removed: "MURATA GQM"
- moved on the sheet: C30, C31, C32, C33, C34, C35, C36, C37, FB2
