File: Notes.kicad_sch (KiCad schematic)
At the start: 0 parts

Commit message: CANFD Power Supply
Changed lines of the file:
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@@
 		(company "Peter Hancak")
 	)
-	(text_box "CONTROLLED IMPEDANCE TRACE WIDTHS\n(Simulations done using ADS Controlled Impedance Line Designer)\n- Simulated is JLCPCB: JLC04161H-3313(Finished thickness1.56mm±10%)\n\n1. Microstrip Edge Coupled, 100 Ohm Differential Impedance, 0.35mm (center to center), 50mmm Length, f=1Ghz, Width = 0.1225 mm\n2. Coplanar Edge Coupled, 100 Ohm Differential Impedance, 0.35mm (center to center), 0.25mm Clearance, 50mmm Length, f=1Ghz, Width = 0.1354 mm, 0.35 - 0.1354 = 0.2146 mm (edge to edge spacing)\n3. USB Coplanar Edge Coupled, 90 Ohm Differential Impedance, 0.5mm (center to center), 0.25mm Clearance, 50mmm Length, f=240Mhz, Width = 0.1704 mm, 0.5 - 0.1704 = 0.3296 mm\n4. USB Microstrip Edge Coupled, 90 Ohm Differential Impedance, 0.5mm (center to center), 50mmm Length, f=240Mhz, Width = 0.1722 mm\n\nRF TRACE 50 Ohm\n- Coplanar single-ended , f is 2.5 GHz, L 20mm, Clearance 0.25mm, Width = 0.1472 mm\n- Coplanar single-ended , f is 5 GHz, L 20mm, Clearance 0.25mm, Width = 0.1475 mm\n\n\nSMA CONNECTOR SIGNAL PIN (MIDDLE) FOOTPRINT\n- With normal 0.35 mm clearance resulted in a veryy significant signal degradation\n- I recalculated the clearance for the middle pin using ADS:\n  - Coplanar Single-Ended, Length: 5mm, Width: 1.37 mmm (width of the pin), f: 5GHz, Clearance = 0.4046 mm\n\nESP32C5 DESIGN CONSIDERATIONS:\n- Flash memory traces NOT length matched. (at 80 MHz not needed)\n- Isolate the CLK trace on the ext flash memory bus\n\nCAN-FD INTERFACE:\n- Traces CANH, CANL impedance matched to 120 Ohm\n- 120 Ohm shunted across CANH and CANL (to be done on the receiver and sender) \n\nSERIES TERMINATION\n- CSI, DSI, SDIO (near P4), UART0, UART1, NOT I2C\nSDIO\n- Array Series termination on SDIO DATA 0-3\n- Individual series termination on CLK, CMD\n- PU on the SDIO INT (Interrupt) pin (Open Drain)"
+	(text_box "CONTROLLED IMPEDANCE TRACE WIDTHS\n(Simulations done using ADS Controlled Impedance Line Designer)\n- Simulated is JLCPCB: JLC04161H-3313(Finished thickness1.56mm±10%)\n\n1. Microstrip Edge Coupled, 100 Ohm Differential Impedance, 0.35mm (center to center), 50mmm Length, f=1Ghz, Width = 0.1225 mm\n2. Coplanar Edge Coupled, 100 Ohm Differential Impedance, 0.35mm (center to center), 0.25mm Clearance, 50mmm Length, f=1Ghz, Width = 0.1354 mm, 0.35 - 0.1354 = 0.2146 mm (edge to edge spacing)\n3. USB Coplanar Edge Coupled, 90 Ohm Differential Impedance, 0.5mm (center to center), 0.25mm Clearance, 50mmm Length, f=240Mhz, Width = 0.1704 mm, 0.5 - 0.1704 = 0.3296 mm\n4. USB Microstrip Edge Coupled, 90 Ohm Differential Impedance, 0.5mm (center to center), 50mmm Length, f=240Mhz, Width = 0.1722 mm\n\nRF TRACE 50 Ohm\n- Coplanar single-ended , f is 2.5 GHz, L 20mm, Clearance 0.25mm, Width = 0.1472 mm\n- Coplanar single-ended , f is 5 GHz, L 20mm, Clearance 0.25mm, Width = 0.1475 mm\n\n\nSMA CONNECTOR SIGNAL PIN (MIDDLE) FOOTPRINT\n- With normal 0.35 mm clearance resulted in a veryy significant signal degradation\n- I recalculated the clearance for the middle pin using ADS:\n  - Coplanar Single-Ended, Length: 5mm, Width: 1.37 mmm (width of the pin), f: 5GHz, Clearance = 0.4046 mm\n\nESP32C5 DESIGN CONSIDERATIONS:\n- Flash memory traces NOT length matched. (at 80 MHz not needed)\n- Isolate the CLK trace on the ext flash memory bus\n\nCAN-FD INTERFACE:\n- Two parallel CAN-FD interfaces in the single connector (each row)\n- 120 Ohm shunted across CANH and CANL (to be done on the receiver and sender) \n- A 10u capacitor has been added on the shield pins.\n  - Both shield pins connected\n  - Capacitor is to be replaced by GND jumper at primary node \n\nSERIES TERMINATION\n- CSI, DSI, SDIO (near P4), UART0, UART1, NOT I2C\nSDIO\n- Array Series termination on SDIO DATA 0-3\n- Individual series termination on CLK, CMD\n- PU on the SDIO INT (Interrupt) pin (Open Drain)"
 		(exclude_from_sim no)
 		(at 113.03 29.464 0)

Commit message: C5 RF Update
Changed lines of the file:
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@@
 		(exclude_from_sim no)
 		(at 113.03 29.464 0)
-		(size 73.152 128.905)
+		(size 73.152 73.406)
 		(margins 0.75 0.75 0.75 0.75)
 		(stroke
+			(width 0)
+			(type dash)
+		)
+		(fill
+			(type none)
+		)
+		(effects
+			(font
+				(size 1 1)
+			)
+			(justify left top)
+		)
+	)
+	(text_box "VDDA1, VDDA2 DESIGN\nSwitching from 0201 to 0402 components for hand-soldering is a practical choice. The main trade-off is that 0402 components have slightly higher Equivalent Series Inductance (L \nESL\n​	\n ≈0.4 nH−0.5 nH compared to ∼0.2 nH for 0201).\nAt a 1.3 mm trace distance, combining the larger 0402 component body with the trace and via parasitics raises the total loop inductance (L \ntotal\n​	\n ) to roughly 1.4 nH−1.6 nH.\nRecommended 0402 Capacitor Tuning\nTo maintain the minimum impedance notch in the 5.18 GHz - 5.88 GHz Wi-Fi 6 band with L \ntotal\n​	\n ≈1.5 nH, you need a lower total capacitance value (C \ntotal\n​	\n ≈0.5 pF−0.6 pF).\n1. Two Parallel 0402 Capacitors (Recommended Configuration)\nValue: Two 0.27 pF or 0.3 pF 0402 (C0G/NP0) capacitors in parallel.\nEffective Capacitance: C \ntotal\n​	\n ≈0.54 pF−0.60 pF.\nTarget Resonant Frequency:\nf \n0\n​	\n = \n2π \n1.5 nH×0.56 pF\n\n​	\n \n1\n​	\n ≈5.48 GHz\nWhy it works well for hand-soldering: 0402 footprints are far easier to rework with a fine conical or chisel tip. Placing two 0402 pads in parallel cuts the 0402 package body inductance in half down to ∼0.22 nH, matching 0201 high-frequency performance.\n2. Single 0402 Capacitor (Alternative)\nValue: One 0.5 pF or 0.56 pF 0402 (C0G/NP0) capacitor.\nEffective Capacitance: C \ntotal\n​	\n ≈0.5 pF−0.56 pF.\nTrade-off: A single 0402 pad takes up less layout area near the pin, but has slightly higher net inductance than two parallel pads.\nLayout Steps for Hand-Soldered 0402 RF Bypass\n1\nWiden the Connection Neck\nLowers trace inductance\nRoute a wide copper neck of 16-20 mil (0.4 mm−0.5 mm) for the 1.3 mm distance leading from the 0402 pads to the VDDA pin.\nVerification: A wider neck offsets the extra L \nESL\n​	\n  of the larger 0402 footprint body.\n\n2\nAdd Parallel Via Stitching\nCuts via return loop\nPlace two dedicated ground vias immediately adjacent to the ground pads of the 0402 capacitors, dropping directly down to the Layer 2 ground plane.\nVerification: Multi-via grounding keeps ground return inductance below 0.1 nH.\n\n3\nExtend Pad Landings Slightly\nHand-soldering optimization\nIn your PCB CAD tool, extend the outer edges of the 0402 pads by 0.1 mm - 0.2 mm to provide a small toe fillet for your soldering iron tip and solder wire.\nVerification: Good solder fillets ensure low DC and RF contact resistance at the termination joint.\n\nComponent Specification Summary\n\nComponent,Quantity & Size,Dielectric,Recommended Values,Expected Resonant Notch\nDual 0402 (Best),2× 0402,C0G / NP0 (±0.05 pF or ±0.1 pF),0.27 pF or 0.3 pF,5.3 GHz - 5.8 GHz\nSingle 0402,1× 0402,C0G / NP0 (±0.05 pF or ±0.1 pF),0.5 pF or 0.56 pF,5.2 GHz - 5.7 GHzComponent,Quantity & Size,Dielectric,Recommended Values,Expected Resonant Notch\nDual 0402 (Best),2× 0402,C0G / NP0 (±0.05 pF or ±0.1 pF),0.27 pF or 0.3 pF,5.3 GHz - 5.8 GHz\nSingle 0402,1× 0402,C0G / NP0 (±0.05 pF or ±0.1 pF),0.5 pF or 0.56 pF,5.2 GHz - 5.7 GHz"
+		(exclude_from_sim no)
+		(at 113.03 107.95 0)
+		(size 73.152 143.1739)
+		(margins 0.75 0.75 0.75 0.75)
+		(stroke
