File: ESP32-P4NRW16_Power.kicad_sch (KiCad schematic)
At the start: 36 parts, among them U1 ESP32-P4NRW16

Commit message: Interface Update
Parts:
- removed TP1, TP2, TP3, TP4: TestPoint, TestPoint:TestPoint_Pad_1.5x1.5mm, symbol Connector:TestPoint
Other:
- note removed: "Low-Power (LP) Core and Always-On (AON) Domain"
- note removed: "To Power Flash chip 1V8/3V3(Flash)"
- company: (none) -> Peter Hancak
- title: (none) -> ESP32P4C5_BOARD
