File: CAN-FD_BUS.kicad_sch (KiCad schematic)
At the start: 10 parts, among them IC2 CAN_MCP2518FDT-H_SL, IC3 CAN_ATA6563-GAQW1, Y1 Crystal_ABM8G-40.000MHZ-18-D2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

Commit message: Interface Update
Parts:
- IC2: value CAN_MCP2518FDT-H_SL -> XINLUDA XLP2518FDT/ESL
Other:
- note added: "CAN_MCP2518FDT-H_SL"
- company: (none) -> Peter Hancak
- title: (none) -> ESP32P4C5_BOARD
Changed lines of the file:
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@@
 	(generator_version "8.0")
 	(paper "A4")
+	(title_block
+		(title "ESP32P4C5_BOARD")
+		(date "2026-06-01")
+		(rev "A")
+		(company "Peter Hancak")
+	)
 	(junction
 		(at 175.26 107.95)
@@
 			(font
 				(size 1.27 1.27)
+			)
+		)
+	)
+	(text "CAN_MCP2518FDT-H_SL\n"
+		(exclude_from_sim no)
+		(at 154.432 81.788 0)
+		(effects
+			(font
+				(size 1 1)
 			)
 		)
@@
 			)
 		)
-		(property "Value" "CAN_MCP2518FDT-H_SL"
-			(at 152.908 79.502 0)
+		(property "Value" "XINLUDA XLP2518FDT/ESL"
+			(at 154.178 79.248 0)
 			(effects
 				(font
@@
 		(dnp no)
 		(property "Reference" "Y1"
-			(at 148.6214 82.55 0)
-			(effects
-				(font
+			(at 151.13 104.648 90)
+			(effects
+				(font

Commit message: Power Rail Update
Connections:
- net CANH renamed CAN+
- net CANL renamed CAN-
Changed lines of the file:
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@@
 		)
 	)
-	(label "CANL"
+	(label "CAN-"
 		(at 223.52 99.06 180)
 		(effects
@@
 		)
 	)
-	(label "CANH"
+	(label "CAN+"
 		(at 223.52 87.63 180)
 		(effects
