File: CAN-FD_BUS.kicad_sch (KiCad schematic)
At the start: 10 parts, among them IC2 XINLUDA XLP2518FDT/ESL, IC3 CAN_ATA6563-GAQW1, Y1 Crystal_ABM8G-40.000MHZ-18-D2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

Commit message: ESP32P4_Fix
Parts:
- removed JST1: JST_S3B-XH-2.54, Personal_Project:JST_S3B-XH-SHDRRA3W64P0X250_1X3_990X1150X610P, symbol Personal_Projects:JST_S3B-XH-A-1_LF_SN
- added J4: CAN_HDR, Connector_PinHeader_2.54mm:PinHeader_1x03_P2.54mm_Horizontal, symbol Connector_Generic:Conn_01x03
Connections:
- net CAN+: now also J4.3 (Pin_3)
- net CAN-: now also J4.2 (Pin_2)
- net GND: now also J4.1 (Pin_1)

Commit message: CANFD Power Supply
Parts:
- removed J4: CAN_HDR, Connector_PinHeader_2.54mm:PinHeader_1x03_P2.54mm_Horizontal, symbol Connector_Generic:Conn_01x03
- removed R3: 120R, Resistor_SMD:R_0603_1608Metric, symbol Device:R
- added C79: 10n_500V, Capacitor_SMD:C_0805_2012Metric, symbol Device:C
- added DI1: Diode_PESD2CANFD24L-TR, Package_TO_SOT_SMD:SOT-23, symbol Personal_Components:Diode_PESD5V0U2BT-Q
- added J11: CAN_OUT_HDR, Connector_PinHeader_2.54mm:PinHeader_2x04_P2.54mm_Horizontal, symbol Connector_Generic:Conn_02x04_Odd_Even
- added R50: 120R, Resistor_SMD:R_0603_1608Metric, symbol Device:R
Connections:
- net GND: now also C79.1, DI1.3 (CC), J11.3 (Pin_3), J11.4 (Pin_4)
- net CAN+ renamed CANH
- net CANH: now also DI1.2 (K2), J11.5 (Pin_5), J11.6 (Pin_6), R50.1
- net CAN- renamed CANL
- net CANL: now also DI1.1 (K1), J11.7 (Pin_7), J11.8 (Pin_8), R50.2
- new net: C79.2, J11.1 (Pin_1), J11.2 (Pin_2)
Other:
- note added: "Differential Impedance: 120 Ohm"
- note added: "OPTIOAL - ONLY ADD ON TERMINAL NODE"
- note added: "Reference board has first pin unconnected"
- note added: "To connect the cable shield - To GND on primary node - To GND through 10n Capacitor on secondary nodes"
- moved on the sheet: C17, C28, C38, C39, C9, IC2, IC3, Y1
