File: Interface_DSI_CSI.kicad_sch (KiCad schematic)
At the start: 3 parts

Commit message: Readme updated
Parts:
- removed FPC3: FPC_40PIN, Personal_Project:FPC_AMPHENOL_10051922-3010ELF, symbol Personal_Projects:FPC_40PIN
Connections:
- no-connect marks 5 -> 4
Other:
- note removed: "IMO=0 interface mode select. MIPI"
- note removed: "IMO=1 interface mode select MIPI"
