File: ESP32P4C5_Board.kicad_sch (KiCad schematic)
At the start: 0 parts

Commit message: Readme updated
Connections:
- no-connect marks 6 -> 12
Other:
- sheet Interface_DSI_CSI ports: added none; removed DSI_CLKN, DSI_CLKP, DSI_D0N, DSI_D0P, DSI_D1N, DSI_D1P, DSI_LEDA, DSI_LEDK, DSI_RESET

Commit message: PCB Layout PDF
Connections:
- no-connect marks 12 -> 13
Other:
- sheet ESP32-P4NRW16 ports: added DSI_REXT; removed none
