File: ESP32P4C5_Board.kicad_sch (KiCad schematic)
At the start: 0 parts

Commit message: RF_Layout
Other:
- added sheet ESP32-C5HR8_RF (vESP32-C5HR8_RF.kicad_sch)
- sheet ESP32-C5HR8 ports: added ANT_2G_M, ANT_5G_M; removed none
Changed lines of the file:
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@@
+	(wire
+		(pts
+			(xy 263.652 59.69) (xy 271.78 59.69)
+		)
+		(stroke
+			(width 0)
+			(type default)
+		)
+	)
 	(wire
 		(pts
@@
 	(wire
 		(pts
+			(xy 263.652 57.15) (xy 274.32 57.15)
+		)
+		(stroke
+			(width 0)
+			(type default)
+		)
+	)
+	(wire
+		(pts
 			(xy 177.546 29.21) (xy 220.98 29.21)
 		)
@@
 	(wire
 		(pts
+			(xy 274.32 147.32) (xy 262.89 147.32)
+		)
+		(stroke
+			(width 0)
+			(type default)
+		)
+	)
+	(wire
+		(pts
 			(xy 133.35 77.47) (xy 80.01 77.47)
 		)
@@
 	(wire
 		(pts
+			(xy 274.32 57.15) (xy 274.32 147.32)
+		)
+		(stroke
+			(width 0)
+			(type default)
+		)
+	)
+	(wire
+		(pts
+			(xy 271.78 149.86) (xy 262.89 149.86)
+		)
+		(stroke
+			(width 0)
+			(type default)
+		)
+	)
+	(wire
+		(pts
 			(xy 111.76 161.29) (xy 217.17 161.29)
 		)
@@
 		(pts
 			(xy 213.36 73.66) (xy 220.726 73.66)
+		)
+		(stroke
+			(width 0)
+			(type default)
+		)
+	)
+	(wire
+		(pts
+			(xy 271.78 59.69) (xy 271.78 149.86)
 		)
 		(stroke
@@
 			(project "ESP32P4C5_Board"
 				(path "/d4a17687-8854-438f-9913-a6ddcff1a679"
-					(page "8")
+					(page "10")
 				)
 			)
@@
 			(project "ESP32P4C5_Board"
 				(path "/d4a17687-8854-438f-9913-a6ddcff1a679"
-					(page "7")
+					(page "8")
 				)
 			)
@@
 			(project "ESP32P4C5_Board"
 				(path "/d4a17687-8854-438f-9913-a6ddcff1a679"
-					(page "10")
+					(page "11")
+				)
+			)
+		)
+	)
+	(sheet
+		(at 220.98 143.51)
+		(size 41.91 12.7)
+		(exclude_from_sim no)
+		(in_bom yes)
+		(on_board yes)
+		(dnp no)
+		(fields_autoplaced yes)
+		(stroke
+			(width 0.1524)
+			(type solid)
+		)
+		(fill
+			(color 0 255 255 1)
+		)
+		(property "Sheetname" "ESP32-C5HR8_RF"
+			(at 220.98 142.7984 0)
+			(show_name no)
+			(do_not_autoplace no)
+			(effects
+				(font
+					(size 1.27 1.27)
+				)
+				(justify left bottom)
+			)
+		)
+		(property "Sheetfile" "vESP32-C5HR8_RF.kicad_sch"
+			(at 220.98 156.7946 0)
+			(show_name no)
+			(do_not_autoplace no)
+			(effects
+				(font
+					(size 1.27 1.27)
+				)
+				(justify left top)
+			)
+		)
+		(pin "ANT_2G_M" bidirectional
+			(at 262.89 147.32 0)
+			(effects
+				(font
+					(size 1.27 1.27)
+				)
+				(justify right)
+			)
+		)
+		(pin "ANT_5G_M" bidirectional
+			(at 262.89 149.86 0)
+			(effects
+				(font
+					(size 1.27 1.27)
+				)
+				(justify right)
+			)
+		)
+		(instances
+			(project "ESP32P4C5_Board"
+				(path "/d4a17687-8854-438f-9913-a6ddcff1a679"
+					(page "7")
 				)
 			)
@@
 			)
 		)
+		(pin "ANT_2G_M" bidirectional
+			(at 263.652 57.15 0)
+			(effects
+				(font
+					(size 1.27 1.27)
+				)
+				(justify right)
+			)
+		)
+		(pin "ANT_5G_M" bidirectional
+			(at 263.652 59.69 0)
+			(effects
+				(font
+					(size 1.27 1.27)
+				)
+				(justify right)
+			)
+		)
 		(instances
 			(project "ESP32P4C5_Board"
@@
 	(sheet
 		(at 220.98 104.902)
-		(size 42.164 53.34)
+		(size 42.164 32.258)
 		(exclude_from_sim no)
 		(in_bom yes)
@@
 		)
 		(property "Sheetfile" "Interfaces.kicad_sch"
-			(at 220.98 158.8266 0)
+			(at 220.98 137.7446 0)
 			(show_name no)
 			(do_not_autoplace no)
