File: ESP32-P4NRW16.kicad_sch (KiCad schematic)
At the start: 35 parts, among them J1 P4_DEBUG_PINS, SW1 XUNPU DSHP-01-TS-GER, U1 ESP32-P4NRW16, U11 BY25Q128ESSIG(T), U15 SN74LVC1G07DBVR, Y2 ECS-400-10-33B-CKM-TR

Commit message: Readme updated
Other:
- note removed: "------ MUST SELECT AVAILABLE FLASH"
Changed lines of the file:
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@@
-		)
-	)
-	(text "------ MUST SELECT AVAILABLE FLASH"
-		(exclude_from_sim no)
-		(at 15.748 101.6 0)
-		(effects
-			(font
-				(size 1.27 1.27)
-			)
 		)
 	)

Commit message: PCB Layout PDF
Parts:
- removed R2: 4k02, Resistor_SMD:R_0603_1608Metric, symbol Device:R
Changed lines of the file:
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@@
 	(wire
 		(pts
-			(xy 250.19 81.28) (xy 254 81.28)
-		)
-		(stroke
-			(width 0)
-			(type default)
-		)
-	)
-	(wire
-		(pts
 			(xy 207.01 73.66) (xy 180.34 73.66)
 		)
@@
 	(wire
 		(pts
-			(xy 180.34 81.28) (xy 242.57 81.28)
+			(xy 180.34 81.28) (xy 207.01 81.28)
 		)
 		(stroke
@@
 		)
 	)
+	(hierarchical_label "DSI_REXT"
+		(shape bidirectional)
+		(at 207.01 81.28 0)
+		(effects
+			(font
+				(size 1.27 1.27)
+			)
+			(justify left)
+		)
+	)
 	(hierarchical_label "GPIO49_PARLIO"
 		(shape input)
@@
 	)
 	(symbol
-		(lib_id "power:GND")
-		(at 254 81.28 90)
-		(mirror x)
-		(unit 1)
-		(body_style 1)
-		(exclude_from_sim no)
-		(in_bom yes)
-		(on_board yes)
-		(in_pos_files yes)
-		(dnp no)
-		(fields_autoplaced yes)
-		(property "Reference" "#PWR031"
-			(at 260.35 81.28 0)
-			(hide yes)
-			(show_name no)
-			(do_not_autoplace no)
-			(effects
-				(font
-					(size 1.27 1.27)
-				)
-			)
-		)
-		(property "Value" "GND"
-			(at 255.2699 78.74 0)
-			(hide yes)
-			(show_name no)
-			(do_not_autoplace no)
-			(effects
-				(font
-					(size 1.27 1.27)
-				)
-				(justify right)
-			)
-		)
-		(property "Footprint" ""
-			(at 254 81.28 0)
-			(hide yes)
-			(show_name no)
-			(do_not_autoplace no)
-			(effects
-				(font
-					(size 1.27 1.27)
-				)
-			)
-		)
-		(property "Datasheet" ""
-			(at 254 81.28 0)
-			(hide yes)
-			(show_name no)
-			(do_not_autoplace no)
-			(effects
-				(font
-					(size 1.27 1.27)
-				)
-			)
-		)
-		(property "Description" "Power symbol creates a global label with name \"GND\" , ground"
-			(at 254 81.28 0)
-			(hide yes)
-			(show_name no)
-			(do_not_autoplace no)
-			(effects
-				(font
-					(size 1.27 1.27)
-				)
-			)
-		)
-		(pin "1"
-		)
-		(instances
-			(project "ESP32P4C5_Board"
-				(path "/d4a17687-8854-438f-9913-a6ddcff1a679/05efe0cf-c24a-4029-900a-f931e619b6bb"
-					(reference "#PWR031")
-					(unit 1)
-				)
-			)
-		)
-	)
-	(symbol
 		(lib_id "Device:R_Pack04")
 		(at 213.36 121.92 90)
@@
 					(unit 1)
 				)
-			)
-		)
-	)
-	(symbol
-		(lib_id "Device:R")
-		(at 246.38 81.28 90)
-		(unit 1)
-		(body_style 1)
-		(exclude_from_sim no)
-		(in_bom yes)
-		(on_board yes)
-		(in_pos_files yes)
-		(dnp no)
-		(property "Reference" "R2"
-			(at 243.332 80.01 90)
-			(show_name no)
-			(do_not_autoplace no)
-			(effects
-				(font
-					(size 1.27 1.27)
-				)
-				(justify left)
-			)
-		)
-		(property "Value" "4k02"
-			(at 254.254 80.01 90)
-			(show_name no)
-			(do_not_autoplace no)
-			(effects
-				(font
-					(size 1.27 1.27)
-				)
-				(justify left)
-			)
-		)
-		(property "Footprint" "Resistor_SMD:R_0603_1608Metric"
-			(at 246.38 83.058 90)
-			(hide yes)
-			(show_name no)
-			(do_not_autoplace no)
-			(effects
-				(font
-					(size 1.27 1.27)
-				)
-			)
-		)
-		(property "Datasheet" ""
-			(at 246.38 81.28 0)
-			(hide yes)
-			(show_name no)
-			(do_not_autoplace no)
-			(effects
-				(font
-					(size 1.27 1.27)
-				)
-			)
-		)
-		(property "Description" "Resistor"
-			(at 246.38 81.28 0)
-			(hide yes)
-			(show_name no)
-			(do_not_autoplace no)
-			(effects
-				(font
-					(size 1.27 1.27)
-				)
-			)
-		)
-		(pin "2"
-		)
-		(pin "1"
-		)
-		(instances
-			(project "ESP32P4C5_Board"
-				(path "/d4a17687-8854-438f-9913-a6ddcff1a679/05efe0cf-c24a-4029-900a-f931e619b6bb"
-					(reference "R2")
-					(unit 1)
-				)

Commit message: VDD_HP_1 Update
Parts:
- removed U1: ESP32-P4NRW16, Personal_Project:ESP32-P4NRW16, symbol Personal_Projects:ESP32-P4NRW16
- added U3: ESP32-P4NRW32X, Personal_Project:ESP32-P4NRW16, symbol Personal_Components:ESP32-P4NRW32X
Connections:
- net CHIP_PU: now also U3.103 (CHIP_PU)
- net CSI_CLKN: now also U3.45 (CSI_CLKN)
- net CSI_CLKP: now also U3.44 (CSI_CLKP)
- net CSI_DATAN0: now also U3.42 (CSI_DATAN0)
- net CSI_DATAN1: now also U3.46 (CSI_DATAN1)
- net CSI_DATAP0: now also U3.43 (CSI_DATAP0)
- net CSI_DATAP1: now also U3.47 (CSI_DATAP1)
- net CSI_REXT: now also U3.48 (CSI_REXT)
- net DSI_CLKN: now also U3.37 (DSI_CLKN)
- net DSI_CLKP: now also U3.38 (DSI_CLKP)
- net DSI_DATAN0: now also U3.40 (DSI_DATAN0)
- net DSI_DATAN1: now also U3.36 (DSI_DATAN1)
- net DSI_DATAP0: now also U3.39 (DSI_DATAP0)
- net DSI_DATAP1: now also U3.35 (DSI_DATAP1)
- net DSI_REXT: now also U3.34 (DSI_REXT)
- net EN_DCDC: now also U3.79 (EN_DCDC)
- net FB_DCDC: now also U3.78 (FB_DCDC)
- net FLASH_CK: now also U3.32 (FLASH_CK)
- net FLASH_CS: now also U3.27 (FLASH_CS)
- net FLASH_D: now also U3.33 (FLASH_D)
- net FLASH_HOLD: now also U3.31 (FLASH_HOLD)
- net FLASH_Q: now also U3.28 (FLASH_Q)
- net FLASH_WP: now also U3.29 (FLASH_WP)
- net GND: now also U3.105 (GND)
- net GPIO0: now also U3.104 (GPIO0)
- net GPIO1: now also U3.1 (GPIO1)
- net GPIO11: now also U3.12 (GPIO11_SPI2_WP)
- net GPIO12: now also U3.13 (GPIO12)
- net GPIO13: now also U3.14 (GPIO13)
- net GPIO14: now also U3.15 (GPIO14)
- net GPIO15: now also U3.16 (GPIO15)
- net GPIO16: now also U3.17 (GPIO16)
- net GPIO17: now also U3.18 (GPIO17)
- net GPIO18: now also U3.19 (GPIO18)
- net GPIO19: now also U3.20 (GPIO19)
- net GPIO20_SPI_MOSI: now also U3.22 (GPIO20)
- net GPIO21_SPI_MISO: now also U3.23 (GPIO21)
- net GPIO22_SPI_CLK: now also U3.24 (GPIO22)
- net GPIO23_SPI_CS: now also U3.25 (GPIO23)
- net GPIO26_PARLIO_R: now also U3.55 (GPIO26)
- net GPIO27_PARLIO_R: now also U3.56 (GPIO27)
- net GPIO28_PARLIO_R: now also U3.57 (GPIO28)
- net GPIO29_PARLIO_R: now also U3.58 (GPIO29)
- net GPIO2_MTCK: now also U3.2 (GPIO2_MTCK)
- net GPIO30_PARLIO_R: now also U3.60 (GPIO30)
- net GPIO31_PARLIO_R: now also U3.61 (GPIO31)
- net GPIO32_PARLIO_R: now also U3.63 (GPIO32)
- net GPIO33_PARLIO_R: now also U3.64 (GPIO33)
- net GPIO34_BOOTM: now also U3.65 (GPIO34_BOOTM)
- net GPIO35_BOOTM: now also U3.66 (GPIO35_BOOTM)
- net GPIO36_BOOTM: now also U3.68 (GPIO36_BOOTM)
- net GPIO37_BOOTM_UART0_TXD: now also U3.69 (GPIO37_BOOTM)
- net GPIO38_BOOTM_UART0_RXD: now also U3.70 (GPIO38_BOOTM)
- net GPIO39_CDATA0_R: now also U3.80 (GPIO39)
- net GPIO3_MTDI: now also U3.3 (GPIO3_MTDI)
- net GPIO40_CDATA1_R: now also U3.81 (GPIO40)
- net GPIO41_CDATA2_R: now also U3.82 (GPIO41)
- net GPIO42_CDATA3_R: now also U3.83 (GPIO42)
- net GPIO43_CCLK_R: now also U3.84 (GPIO43)
- net GPIO44_CCMD_R: now also U3.86 (GPIO44)
- net GPIO45_CINT: now also U3.87 (GPIO45)
- net GPIO46: now also U3.88 (GPIO46)
- net GPIO47_PARLIO_R: now also U3.89 (GPIO47)
- net GPIO48_PARLIO_R: now also U3.90 (GPIO48)
- net GPIO49_PARLIO_R: now also U3.92 (GPIO49)
- net GPIO4_MTMS: now also U3.4 (GPIO4_MTMS)
- net GPIO50: now also U3.93 (GPIO50)
- net GPIO51: now also U3.94 (GPIO51)
- net GPIO52: now also U3.95 (GPIO52)
- net GPIO53: now also U3.97 (GPIO53)
- net GPIO54: now also U3.98 (GPIO54)
- net GPIO5_MTDO: now also U3.5 (GPIO5_MTDO)
- net GPIO6: now also U3.6 (GPIO6_SPI2_HOLD)
- net P4_USB_HS_DN: now also U3.49 (DM)
- net P4_USB_HS_DP: now also U3.50 (DP)
- net SPI2_CK: now also U3.10 (GPIO9_SPI2_CK)
- net SPI2_CS: now also U3.7 (GPIO7_SPI2_CS)
- net SPI2_MISO: now also U3.11 (GPIO10_SPI2_MISO)
- net SPI2_MOSI: now also U3.8 (GPIO8_SPI2_MOSI)
- net USB1P1_R_N: now also U3.52 (GPIO24_USB1P1_N0)
- net USB1P1_R_P: now also U3.53 (GPIO25_USB1P1_P0)
- net XTAL_N: now also U3.99 (XTAL_N)
- net XTAL_P: now also U3.100 (XTAL_P)

Commit message: PCB Layout Update
Connections:
- net GND: no longer RN5.2 (R2.1), RN5.3 (R3.1), RN5.6 (R3.2), RN5.7 (R2.2)
- net GPIO43_CCLK: now also RN5.7 (R2.2); no longer RN5.8 (R1.2)
- net GPIO43_CCLK_R: now also RN5.2 (R2.1); no longer RN5.1 (R1.1)
- no-connect marks 1 -> 5
Changed lines of the file:
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@@
 	)
 	(junction
-		(at 232.41 132.08)
-		(diameter 0)
-		(color 0 0 0 0)
-	)
-	(junction
 		(at 278.13 129.54)
 		(diameter 0)
@@
 	)
 	(junction
-		(at 219.71 132.08)
-		(diameter 0)
-		(color 0 0 0 0)
-	)
-	(junction
 		(at 44.45 115.57)
 		(diameter 0)
@@
 	)
 	(no_connect
+		(at 220.98 132.08)
+	)
+	(no_connect
 		(at 50.8 35.56)
 	)
+	(no_connect
+		(at 231.14 127)
+	)
+	(no_connect
+		(at 231.14 132.08)
+	)
+	(no_connect
+		(at 220.98 127)
+	)
 	(wire
 		(pts
@@
 	(wire
 		(pts
-			(xy 232.41 129.54) (xy 232.41 132.08)
-		)
-		(stroke
-			(width 0)
-			(type default)
-		)
-	)
-	(wire
-		(pts
 			(xy 270.51 129.54) (xy 278.13 129.54)
 		)
@@
 	(wire
 		(pts
+			(xy 220.98 129.54) (xy 218.44 129.54)
+		)
+		(stroke
+			(width 0)
+			(type default)
+		)
+	)
+	(wire
+		(pts
 			(xy 54.61 125.73) (xy 57.15 125.73)
 		)
@@
 	(wire
 		(pts
-			(xy 232.41 132.08) (xy 231.14 132.08)
-		)
-		(stroke
-			(width 0)
-			(type default)
-		)
-	)
-	(wire
-		(pts
 			(xy 207.01 76.2) (xy 180.34 76.2)
 		)
@@
 	(wire
 		(pts
-			(xy 231.14 129.54) (xy 232.41 129.54)
-		)
-		(stroke
-			(width 0)
-			(type default)
-		)
-	)
-	(wire
-		(pts
 			(xy 180.34 116.84) (xy 208.28 116.84)
 		)
@@
 	(wire
 		(pts
-			(xy 219.71 129.54) (xy 219.71 132.08)
+			(xy 218.44 121.92) (xy 246.38 121.92)
 		)
 		(stroke
@@
 	(wire
 		(pts
-			(xy 218.44 121.92) (xy 246.38 121.92)
+			(xy 111.76 55.88) (xy 134.62 55.88)
 		)
 		(stroke
@@
 	(wire
 		(pts
-			(xy 111.76 55.88) (xy 134.62 55.88)
+			(xy 233.68 129.54) (xy 233.68 127)
 		)
 		(stroke
@@
 	(wire
 		(pts
-			(xy 231.14 127) (xy 246.38 127)
+			(xy 69.85 170.18) (xy 63.5 170.18)
 		)
 		(stroke
@@
 	(wire
 		(pts
-			(xy 69.85 170.18) (xy 63.5 170.18)
+			(xy 278.13 111.76) (xy 278.13 114.3)
 		)
 		(stroke
@@
 	(wire
 		(pts
-			(xy 278.13 111.76) (xy 278.13 114.3)
+			(xy 218.44 129.54) (xy 218.44 127)
 		)
 		(stroke
@@
 	(wire
 		(pts
-			(xy 180.34 127) (xy 220.98 127)
+			(xy 180.34 127) (xy 218.44 127)
 		)
 		(stroke
@@
 	(wire
 		(pts
+			(xy 231.14 129.54) (xy 233.68 129.54)
+		)
+		(stroke
+			(width 0)
+			(type default)
+		)
+	)
+	(wire
+		(pts
 			(xy 265.43 68.58) (xy 257.81 68.58)
 		)
@@
 	(wire
 		(pts
+			(xy 233.68 127) (xy 246.38 127)
+		)
+		(stroke
+			(width 0)
+			(type default)
+		)
+	)
+	(wire
+		(pts
 			(xy 119.38 149.86) (xy 134.62 149.86)
 		)
@@
 	(wire
 		(pts
-			(xy 219.71 132.08) (xy 220.98 132.08)
-		)
-		(stroke
-			(width 0)
-			(type default)
-		)
-	)
-	(wire
-		(pts
 			(xy 104.14 81.28) (xy 96.52 81.28)
 		)
@@
 	(wire
 		(pts
-			(xy 220.98 129.54) (xy 219.71 129.54)
-		)
-		(stroke
-			(width 0)
-			(type default)
-		)
-	)
-	(wire
-		(pts
 			(xy 111.76 96.52) (xy 134.62 96.52)
 		)
@@
 	)
 	(symbol
-		(lib_id "power:GND")
-		(at 219.71 132.08 270)
-		(mirror x)
-		(unit 1)
-		(body_style 1)
-		(exclude_from_sim no)
-		(in_bom yes)
-		(on_board yes)
-		(in_pos_files yes)
-		(dnp no)
-		(fields_autoplaced yes)
-		(property "Reference" "#PWR07"
-			(at 213.36 132.08 0)
-			(hide yes)
-			(show_name no)
-			(do_not_autoplace no)
-			(effects
-				(font
-					(size 1.27 1.27)
-				)
-			)
-		)
-		(property "Value" "GND"
-			(at 218.4401 134.62 0)
-			(hide yes)
-			(show_name no)
-			(do_not_autoplace no)
-			(effects
-				(font
-					(size 1.27 1.27)
-				)
-				(justify right)
-			)
-		)
-		(property "Footprint" ""
-			(at 219.71 132.08 0)
-			(hide yes)
-			(show_name no)
-			(do_not_autoplace no)
-			(effects
-				(font
-					(size 1.27 1.27)
-				)
-			)
-		)
-		(property "Datasheet" ""
-			(at 219.71 132.08 0)
-			(hide yes)
-			(show_name no)
-			(do_not_autoplace no)
-			(effects
-				(font
-					(size 1.27 1.27)
-				)
-			)
-		)
-		(property "Description" "Power symbol creates a global label with name \"GND\" , ground"
-			(at 219.71 132.08 0)
-			(hide yes)
-			(show_name no)
-			(do_not_autoplace no)
-			(effects
-				(font
-					(size 1.27 1.27)
-				)
-			)
-		)
-		(pin "1"
-		)
-		(instances
-			(project "ESP32P4C5_Board"
-				(path "/d4a17687-8854-438f-9913-a6ddcff1a679/05efe0cf-c24a-4029-900a-f931e619b6bb"
-					(reference "#PWR07")
-					(unit 1)
-				)
-			)
-		)
-	)
-	(symbol
 		(lib_id "Device:R_Pack04")
 		(at 212.09 99.06 90)
@@
 					(unit 1)
 				)
-			)
-		)
-	)
-	(symbol
-		(lib_id "power:GND")
-		(at 232.41 132.08 90)
-		(mirror x)
-		(unit 1)
-		(body_style 1)
-		(exclude_from_sim no)
-		(in_bom yes)
-		(on_board yes)
-		(in_pos_files yes)
-		(dnp no)
-		(fields_autoplaced yes)
-		(property "Reference" "#PWR010"
-			(at 238.76 132.08 0)
-			(hide yes)
-			(show_name no)
-			(do_not_autoplace no)
-			(effects
-				(font
-					(size 1.27 1.27)
-				)
-			)
-		)
-		(property "Value" "GND"
-			(at 233.6799 129.54 0)
-			(hide yes)
-			(show_name no)
-			(do_not_autoplace no)
-			(effects
-				(font
-					(size 1.27 1.27)
-				)
-				(justify right)
-			)
-		)
-		(property "Footprint" ""
-			(at 232.41 132.08 0)
-			(hide yes)
-			(show_name no)
-			(do_not_autoplace no)
-			(effects
-				(font
-					(size 1.27 1.27)
-				)
-			)
-		)
-		(property "Datasheet" ""
-			(at 232.41 132.08 0)
-			(hide yes)
-			(show_name no)
-			(do_not_autoplace no)
-			(effects
-				(font
-					(size 1.27 1.27)
-				)
-			)
-		)
-		(property "Description" "Power symbol creates a global label with name \"GND\" , ground"
-			(at 232.41 132.08 0)
-			(hide yes)
-			(show_name no)
-			(do_not_autoplace no)
-			(effects
-				(font
-					(size 1.27 1.27)
-				)
-			)
-		)
-		(pin "1"
-		)
-		(instances
-			(project "ESP32P4C5_Board"
-				(path "/d4a17687-8854-438f-9913-a6ddcff1a679/05efe0cf-c24a-4029-900a-f931e619b6bb"
-					(reference "#PWR010")
-					(unit 1)
-				)
