File: Power_Management.kicad_sch (KiCad schematic)
At the start: 46 parts, among them U6 SMPS_TPS63002DRCR

Commit message: Readme updated
Parts:
- L1: footprint l4 -> Inductor_SMD:L_1008_2520Metric
Changed lines of the file:
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@@
 			)
 		)
-		(property "Footprint" "l4"
+		(property "Footprint" "Inductor_SMD:L_1008_2520Metric"
 			(at 176.53 93.98 0)
 			(hide yes)

Commit message: CANFD Power Supply
Parts:
- removed C40: 100n, Capacitor_SMD:C_0603_1608Metric, symbol Device:C
- removed C44: 10u, Capacitor_SMD:C_0603_1608Metric, symbol Device:C
- removed TP9: TestPoint, TestPoint:TestPoint_Pad_1.5x1.5mm, symbol Connector:TestPoint
- removed U6: SMPS_TPS63002DRCR, Personal_Projects:SMPS_TPS63002DRCR_10-VSON, symbol Personal_Components:SMPS_TPS63002DRCR
- added C45: 2u2, Capacitor_SMD:C_0603_1608Metric, symbol Device:C
- added LDO1: LDO_LDLN050PUR, Package_DFN_QFN:DFN-8-1EP_3x3mm_P0.65mm_EP1.7x2.05mm, symbol Personal_Components:LDO_LDLN050PUR
- added R47, R49: 100k, Resistor_SMD:R_0603_1608Metric, symbol Device:R
- added R48: 316k, Resistor_SMD:R_0603_1608Metric, symbol Device:R
- added U1: TPS61220DCK, Package_TO_SOT_SMD:Texas_R-PDSO-G6, symbol Regulator_Switching:TPS61222DCK
- L3: value 2u2_LPS3015-222MRC -> 4u7_LQH3NPN4R7MMEL; footprint Inductor_SMD:L_Coilcraft_LPS3010 -> Personal_Project:Inductor_LQH3NPN4R7MMEL
- R46: value 100R -> 1M
Connections:
- net L1 is gone; now on net PWR_D+: L3.1
- net GND: now also C45.1, LDO1.4 (GND_1), LDO1.9 (GND_2), R47.2, R49.2, U1.3 (GND)
- net PWR_D+: now also U1.1 (VIN), U1.6 (EN); no longer R46.1
- net 5V+: no longer names the net of C43.2
- net 5V+: now also R46.1, LDO1.5 (EN), LDO1.8 (IN), U1.4 (VOUT)
- net L2: no longer names the net of L3.2
- net L2: now also U1.5 (L)
- net VINA: no longer names the net of R46.2
- net VINA: now also R47.1, U1.2 (FB)
- new net: LDO1.3 (FB), R48.2, R49.1
- new net 5V: C45.2, LDO1.1 (OUT), R48.1
- no-connect marks 3 -> 6
Other:
- note added: "100mV Worst Case Drop"
- note added: "100mV Worst Case Drop (3A, 0.034 Ohm)"
- note added: "PWR+(min) = 3.73 V Worst case + 0.2 V PWR+(min) = 4V aprx."
- note added: "VIN(min) = VOUT+IOUT×(RDS(ON)+DCR VIN(min) = 3.3V+3A x (0.1 Ohm + 0.042 Ohm) VIN(min) = 3.73 V Worst case"
- moved on the sheet: C2, C21, C22, C23, C24, C25, C26, C27, C42, C43, L1, L2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

Commit message: PCB Layout Update
Connections:
- net 5V renamed 5V+
Other:
- note added: "VOUT: 5V5"
Changed lines of the file:
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@@
 		)
 	)
+	(text "VOUT: 5V5"
+		(exclude_from_sim no)
+		(at 91.948 128.27 0)
+		(effects
+			(font
+				(size 1 1)
+			)
+			(justify left)
+		)
+	)
 	(text_box "ON/OFF Switch, Polarity Protection, TVS"
 		(exclude_from_sim no)
@@
 			)
 		)
-		(property "Value" "5V"
-			(at 102.87 165.862 0)
+		(property "Value" "5V+"
+			(at 103.378 165.862 0)
 			(show_name no)
 			(do_not_autoplace no)
