File: USB.kicad_sch (KiCad schematic)
At the start: 12 parts, among them J6 USB_C_Receptacle_USB2.0_16P, J9 USB_C_Receptacle_USB2.0_16P, U2 USBLC6-2SC6, U4 USBLC6-2SC6

Commit message: Update
Parts:
- removed U2, U4: USBLC6-2SC6, Package_TO_SOT_SMD:SOT-23-6, symbol Power_Protection:USBLC6-2SC6
- added U6, U7: DIODE_TPD2E001DZDR, Personal_Projects:DIODE_TPD2E001DZDR, symbol Personal_Components:DIODE_TPD2E001DZDR
Connections:
- net USB_D1+ is gone; now on net USB_DI_D1+: J6.A6 (D+), J6.B6 (D+)
- net USB_D1- is gone; now on net USB_DI_D1-: J6.A7 (D-), J6.B7 (D-)
- net USB_D2+ is gone; now on net USB_DI_D2+: J9.A6 (D+), J9.B6 (D+)
- net USB_D2- is gone; now on net USB_DI_D2-: J9.A7 (D-), J9.B7 (D-)
- net GND: now also U6.1 (GND), U7.1 (GND)
- net USB_DI_D1+: now also U6.3 (IO2)
- net USB_DI_D1-: now also U6.2 (IO1)
- net USB_DI_D2+: now also U7.3 (IO2)
- net USB_DI_D2-: now also U7.2 (IO1)
- net VBUS1+: now also U6.4 (VCC)
- net VBUS2+: now also U7.4 (VCC)
